File: TSOC-USBUART1/revisions/TSOC-BASE-ESP8266-1-0.brd (EAGLE design)
At the start: 45 x 26.4 mm, 39 parts, among them U1 NCP361SNT1G, U2 MIC5219 3.3V, U3 CY7C65213-28PVXI

Commit message: revision 3.1
Parts:
- removed C7: 0.1uF, PatternAgents-ProtoPads:0603-CAP
- removed ESD: SP1001-02JTG, TSOC-ESP8266-BASE:SC70-3
- removed R10: 10K, PatternAgents-ProtoPads:0603-RES
- removed R8, R9: 22, PatternAgents-ProtoPads:0603-RES
- removed U$100: PA_LOGO_SYMMED, PatternAgents-Logos:PA_LOGO_AGENT_MED_SYM
- removed U$101, U$102: TSOC-LOGO-MED, thingSoC:TSOC-LOGO-MED
- added FID4: FIDUCIAL1.5X3, PatternAgents-Misc:FIDUCIAL-1.5X3
- added L1: MH2029-300Y, wuerth-elektronik:0805
- added U$4: TSOC-LOGO-SMALL, thingSoC:TSOC-LOGO-SML
- added U4: CY7C65213-28PVXI, PatternAgents-Cypress:SSOP28DB
- C1: value 470pF -> 2.2uF
- C2: value 2.2uF -> 470pF
- C4: value 470pF -> 1.0uF
- C5: value 1.0uF -> 0.1uF
- R6: value 1M -> 10K
- U$1, U$2: value TSOC-LOGO-MED -> PA_LOGO_SYMMED; device thingSoC:TSOC-LOGO-MED -> PatternAgents-Logos:PA_LOGO_AGENT_MED_SYM
- U$3: value PA_LOGO_SYMMED -> TSOC-LOGO-SMALL; device PatternAgents-Logos:PA_LOGO_AGENT_MED_SYM -> thingSoC:TSOC-LOGO-SML
- U1: value NCP361SNT1G -> NUF2221W1T2; device PatternAgents-OnSemi:SOP95P275X110-5N -> PatternAgents-OnSemi:SOT-363
- U2: value MIC5219 3.3V -> NCP361SNT1G; device SparkFun-PowerIC:SOT23-5 -> PatternAgents-OnSemi:SOP95P275X110-5N
- U3: value CY7C65213-28PVXI -> MIC5219 3.3V; device PatternAgents-Cypress:SSOP28DB -> SparkFun-PowerIC:SOT23-5
- moved FID3 42.4 mm to (1.02, 25.4)
- moved U$1 32.1 mm to (40.9, 2.79)
- moved FID1 23.9 mm to (1.02, 1.02)
- moved U$2 19.3 mm to (40.9, 2.79), flipped to the bottom
- moved U$3 17.2 mm to (34.5, 18.8), flipped to the bottom
- moved R6 16.2 mm to (20.1, 12.7), turned to 0 degrees
- moved C5 13.5 mm to (35.6, 6.10), turned to 180 degrees
- moved R5 12.3 mm to (10.9, 11.4), turned to 90 degrees
- moved R7 12.3 mm to (5.84, 22.6), turned to 0 degrees
- moved U3 11.2 mm to (16.0, 11.7), turned to 270 degrees
- moved U2 8.39 mm to (7.62, 11.4), turned to 0 degrees
- moved C1 7.97 mm to (13.0, 11.4)
- moved C2 7.18 mm to (20.1, 10.4), turned to 0 degrees
- moved U1 4.02 mm to (8.89, 7.62), turned to 270 degrees
- moved C4 3.56 mm to (20.1, 6.86)
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- renumbered JP100 to JP2, JP101 to JP1
Connections:
- net !CTS: now also U4.11; no longer U3.11
- net !DCD: now also U4.10; no longer U3.10
- net !DSR: now also U4.9; no longer U3.9
- net !DTR: now also U4.2; no longer U3.2
- net !POWER: now also U4.14; no longer U3.14
- net !RI: now also U4.6; no longer U3.6
- net !RST: now also R6.2, U4.19; no longer R10.2, U3.19
- net !RTS: now also U4.3; no longer U3.3
- net !RX_LED: now also U4.22; no longer U3.22
- net !SLEEP: now also U4.12; no longer U3.12
- net !TX_LED: now also U4.23; no longer U3.23
- net !USB_FAULT: now also R5.1, U2.4, U3.3; no longer R7.1, U1.4, U2.3
- net 3V3: now also C5.2, R6.1, R7.1, U3.5, U4.4; no longer C7.2, R10.1, R5.1, U2.5, U3.4
- net 5V0: now also C1.1, R5.2, U2.5, U3.1, U4.20; no longer C2.1, R7.2, U1.5, U2.1, U3.20
- net BCD0: now also U4.28; no longer U3.28
- net BCD1: now also U4.27; no longer U3.27
- net BUS_DET: now also R7.2, U4.8; no longer R5.2, U3.8
- net BYPASS: now also C2.1, U3.4; no longer C4.1, U2.4
- net GND: now also C1.2, C4.1, L1.2, U2.3, U3.2, U4.18, U4.21, U4.7; no longer C1.1, C4.2, C7.1, ESD.3, R6.1, U1.3, U3.18, U3.21, U3.7
- net RXD: now also U4.5; no longer U3.5
- net TXD: now also U4.1; no longer U3.1
- net TXDEN: now also U4.13; no longer U3.13
- net USB1_DM: now also U1.1; no longer ESD.2, R9.1
- net USB1_DP: now also U1.3; no longer ESD.1, R8.1
- net USB1_M: now also U1.6, U4.16; no longer R9.2, U3.16
- net USB1_P: now also U1.4, U4.15; no longer R8.2, U3.15
- net USB1_SHIELD: now also L1.1; no longer C1.2, R6.2
- net USB1_VBUS: now also U1.5, U2.1; no longer U1.1
- net VCCD: now also C4.2, U4.17; no longer C5.2, U3.17
Routing:
- net USB1_P: track 7.45 -> 14.2 mm
- net USB1_M: track 8.70 -> 15.3 mm
- net USB1_DP: track 9.92 -> 3.46 mm
- net USB1_DM: track 9.86 -> 3.41 mm
- net GND: track 124.0 -> 119.5 mm, vias 11 -> 10
- net USB1_VBUS: track 7.64 -> 11.5 mm
- net USB1_SHIELD: track 19.4 -> 16.6 mm
- net VCCD: track 3.02 -> 4.43 mm
Other:
- board text added: "Rev3.0"
- board text removed: "1/5/2016"
- board text removed: "Rev3.1"
- board text removed: "TTL UART"
