File: TSOC-USBUART1/revisions/TSOC-BASE-ESP8266-1-0.sch (EAGLE design)
At the start: 37 parts, among them U1 NCP361SNT1G, U2 MIC5219 3.3V, U3 CY7C65213-28PVXI

Commit message: revision 3.1
Parts:
- removed C7: 0.1uF, PatternAgents-ProtoPads:CAP0603-CAP
- removed ESD: SP1001-02JTG, TSOC-ESP8266-BASE:SP1001-02JTG
- removed R10: 10K, PatternAgents-ProtoPads:RESISTOR0603-RES
- removed R8, R9: 22, PatternAgents-ProtoPads:RESISTOR0603-RES
- removed U$101: TSOC-LOGO-MED, thingSoC:TSOC-LOGO-MED
- added FID4: FIDUCIAL1.5X3, PatternAgents-Misc:FIDUCIAL1.5X3
- added L1: MH2029-300Y, wuerth-elektronik:WE-CBF_0805
- added U$4: TSOC-LOGO-SMALL, thingSoC:TSOC-LOGO-SMALL
- added U4: CY7C65213-28PVXI, PatternAgents-Cypress:CY7C65213-28PVXI
- C1: value 470pF -> 2.2uF
- C2: value 2.2uF -> 470pF
- C4: value 470pF -> 1.0uF
- C5: value 1.0uF -> 0.1uF
- R6: value 1M -> 10K
- U$2: value TSOC-LOGO-MED -> PA_LOGO_SYMMED; device thingSoC:TSOC-LOGO-MED -> PatternAgents-Logos:PA_LOGO_SYMMED
- U$3: value PA_LOGO_SYMMED -> TSOC-LOGO-SMALL; device PatternAgents-Logos:PA_LOGO_SYMMED -> thingSoC:TSOC-LOGO-SMALL
- U1: value NCP361SNT1G -> NUF2221W1T2; device PatternAgents-OnSemi:NCP361SNT1G -> PatternAgents-OnSemi:NUF2221W1T2
- U2: value MIC5219 3.3V -> NCP361SNT1G; device SparkFun-PowerIC:V_REG_MIC52193.3V -> PatternAgents-OnSemi:NCP361SNT1G
- U3: value CY7C65213-28PVXI -> MIC5219 3.3V; device PatternAgents-Cypress:CY7C65213-28PVXI -> SparkFun-PowerIC:V_REG_MIC52193.3V
- renumbered JP100 to JP2, JP101 to JP1, U$100 to U$1
Connections:
- net !CTS: now also U4.CTS; no longer U3.CTS
- net !DCD: now also U4.DCD; no longer U3.DCD
- net !DSR: now also U4.DSR; no longer U3.DSR
- net !DTR: now also U4.DTR; no longer U3.DTR
- net !POWER: now also U4.GPIO3; no longer U3.GPIO3
- net !RI: now also U4.RI; no longer U3.RI
- net !RST: now also R6.2, U4.RESET; no longer R10.2, U3.RESET
- net !RTS: now also U4.RTS; no longer U3.RTS
- net !RX_LED: now also U4.GPIO1; no longer U3.GPIO1
- net !SLEEP: now also U4.GPIO4; no longer U3.GPIO4
- net !TX_LED: now also U4.GPIO0; no longer U3.GPIO0
- net !USB_FAULT: now also R5.1, U2.!FLAG, U3.EN; no longer R7.1, U1.!FLAG, U2.EN
- net 3V3: now also C5.2, R6.1, R7.1, U3.OUT, U4.VCCIO; no longer C7.2, R10.1, R5.1, U2.OUT, U3.VCCIO
- net 5V0: now also C1.1, R5.2, U2.OUT, U3.IN, U4.VCC; no longer C2.1, R7.2, U1.OUT, U2.IN, U3.VCC
- net BCD0: now also U4.GPIO7; no longer U3.GPIO7
- net BCD1: now also U4.GPIO6; no longer U3.GPIO6
- net BUS_DET: now also R7.2, U4.GPIO5; no longer R5.2, U3.GPIO5
- net BYPASS: now also C2.1, U3.BP; no longer C4.1, U2.BP
- net GND: now also C1.2, C4.1, L1.2, U2.!EN, U3.GND, U4.GND@18, U4.GND@21, U4.GND@7; no longer C1.1, C4.2, C7.1, ESD.A, R6.1, U1.!EN, U3.GND@18, U3.GND@21, U3.GND@7
- net RXD: now also U4.RXD; no longer U3.RXD
- net TXD: now also U4.TXD; no longer U3.TXD
- net TXDEN: now also U4.GPIO2; no longer U3.GPIO2
- net USB1_DM: now also U1.D1A; no longer ESD.C2, R9.1
- net USB1_DP: now also U1.D2A; no longer ESD.C1, R8.1
- net USB1_M: now also U1.D1B, U4.USBDM; no longer R9.2, U3.USBDM
- net USB1_P: now also U1.D2B, U4.USBDP; no longer R8.2, U3.USBDP
- net USB1_SHIELD: now also L1.1; no longer C1.2, R6.2
- net USB1_VBUS: now also U1.VBUS, U2.IN; no longer U1.IN
- net VCCD: now also C4.2, U4.VCCD; no longer C5.2, U3.VCCD
Other:
- note removed: "3.1"
- moved on the sheet: C1, C2, C4, C5, R5, R6, R7
